File: Hardware/in-out-port/in-out-port/in-out-port.kicad_sch (KiCad schematic)
At the start: 2 parts, among them J1 Debug, U1 STM32G030F6Px

Commit message: updated Schematic
Parts:
- added C1: C, symbol Device:C
Connections:
- net +3.3V: now also U1.4 (VDD)
- net GND: now also J1.4 (Pin_4), U1.5 (VSS)
- net SWCLK: now also J1.3 (Pin_3), U1.18 (PA13)
- net SWDIO: now also J1.2 (Pin_2), U1.19 (PA14/PA15)
- net vm_out_1: now reaches U1.1 (PB7/PB8)
- net cm_out_1: now reaches U1.10 (PA3)
- net out_3: now reaches U1.11 (PA4)
- net cm_out_2: now reaches U1.12 (PA5)
- net out_2: now reaches U1.13 (PA6)
- net cm_out_3: now reaches U1.14 (PA7)
- net out_1: now reaches U1.15 (PB0/PB1/PB2/PA8)
- net rs485-tx: now reaches U1.16 (PA11/PA9)
- net rs485-rx: now reaches U1.17 (PA12/PA10)
- net vm_out_2: now reaches U1.2 (PC14/PB9)
- net rs485-de: now reaches U1.20 (PB3/PB4/PB5/PB6)
- net vm_out_3: now reaches U1.3 (PC15)
- net in_1: now reaches U1.7 (PA0)
- net in_2: now reaches U1.8 (PA1)
- net in_3: now reaches U1.9 (PA2)
Other:
- note added: "PB0 = pwm tim1 PA6 = pwm tim3 PA4 = pwm tim14 PA0 = ADC_in0 PA1 = ADC_in1 PA2 = ADC_in2 PA3 = ADC_in3 PA5 = ADC_in5 PA7 = ADC_in7 PB7 = ADC_in11 PC14 = GPIO_Analog PC15 = GPIO_Analog"
- moved on the sheet: U1
Changed lines of the file:
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@@
 (kicad_sch (version 20230121) (generator eeschema)
   (paper "A3")
+  (wire (pts (xy 164.465 53.975) (xy 164.465 56.515))
+    (stroke (width 0) (type default))
+  )
+  (wire (pts (xy 168.91 25.4) (xy 165.735 25.4))
+    (stroke (width 0) (type default))
+  )
+  (wire (pts (xy 184.785 64.135) (xy 189.23 64.135))
+    (stroke (width 0) (type default))
+  )
+  (wire (pts (xy 165.735 25.4) (xy 165.735 27.305))
+    (stroke (width 0) (type default))
+  )
   (polyline (pts (xy 12.7 78.74) (xy 111.125 78.74))
     (stroke (width 0) (type default))
   )
+  (wire (pts (xy 165.735 22.86) (xy 168.91 22.86))
+    (stroke (width 0) (type default))
+  )
+  (wire (pts (xy 139.7 69.215) (xy 144.145 69.215))
+    (stroke (width 0) (type default))
+  )
+  (wire (pts (xy 184.785 71.755) (xy 189.23 71.755))
+    (stroke (width 0) (type default))
+  )
+  (wire (pts (xy 164.465 97.155) (xy 164.465 99.06))
+    (stroke (width 0) (type default))
+  )
+  (wire (pts (xy 139.7 79.375) (xy 144.145 79.375))
+    (stroke (width 0) (type default))
+  )
+  (wire (pts (xy 184.785 89.535) (xy 188.595 89.535))
+    (stroke (width 0) (type default))
+  )
+  (wire (pts (xy 184.785 66.675) (xy 189.23 66.675))
+    (stroke (width 0) (type default))
+  )
+  (wire (pts (xy 165.735 20.32) (xy 168.91 20.32))
+    (stroke (width 0) (type default))
+  )
+  (wire (pts (xy 139.7 74.295) (xy 144.145 74.295))
+    (stroke (width 0) (type default))
+  )
+  (wire (pts (xy 139.7 66.675) (xy 144.145 66.675))
+    (stroke (width 0) (type default))
+  )
+  (wire (pts (xy 184.785 61.595) (xy 189.23 61.595))
+    (stroke (width 0) (type default))
+  )
   (polyline (pts (xy 111.125 13.335) (xy 111.125 78.74))
     (stroke (width 0) (type default))
   )
+  (wire (pts (xy 184.785 84.455) (xy 189.23 84.455))
+    (stroke (width 0) (type default))
+  )
+  (wire (pts (xy 184.785 74.295) (xy 189.23 74.295))
+    (stroke (width 0) (type default))
+  )
+  (wire (pts (xy 184.785 81.915) (xy 189.23 81.915))
+    (stroke (width 0) (type default))
+  )
+  (wire (pts (xy 184.785 79.375) (xy 189.23 79.375))
+    (stroke (width 0) (type default))
+  )
+  (wire (pts (xy 184.785 76.835) (xy 189.23 76.835))
+    (stroke (width 0) (type default))
+  )
+  (wire (pts (xy 139.7 76.835) (xy 144.145 76.835))
+    (stroke (width 0) (type default))
+  )
+  (wire (pts (xy 184.785 69.215) (xy 189.23 69.215))
+    (stroke (width 0) (type default))
+  )
+  (wire (pts (xy 184.785 86.995) (xy 188.595 86.995))
+    (stroke (width 0) (type default))
+  )
   (text "power supply in max 35V to 3.3V" (at 20.32 74.93 0)
     (effects (font (size 1.27 1.27)) (justify left bottom))
   )
+  (text "PB0 = pwm tim1\nPA6 = pwm tim3\nPA4 = pwm tim14\n\nPA0 = ADC_in0\nPA1 = ADC_in1\nPA2 = ADC_in2\nPA3 = ADC_in3\nPA5 = ADC_in5\nPA7 = ADC_in7\n\nPB7 = ADC_in11\n\nPC14 = GPIO_Analog\nPC15 = GPIO_Analog"
+    (at 127.635 115.57 0)
+    (effects (font (size 1.27 1.27)) (justify left bottom))
+  )
+  (label "rs485-rx" (at 189.23 84.455 0) (fields_autoplaced)
+    (effects (font (size 1.27 1.27)) (justify left bottom))
+  )
+  (label "out_3" (at 189.23 71.755 0) (fields_autoplaced)
+    (effects (font (size 1.27 1.27)) (justify left bottom))
+  )
+  (label "vm_out_1" (at 139.7 79.375 180) (fields_autoplaced)
+    (effects (font (size 1.27 1.27)) (justify right bottom))
+  )
+  (label "out_1" (at 139.7 74.295 180) (fields_autoplaced)
+    (effects (font (size 1.27 1.27)) (justify right bottom))
+  )
+  (label "in_1" (at 189.23 61.595 0) (fields_autoplaced)
+    (effects (font (size 1.27 1.27)) (justify left bottom))
+  )
+  (label "out_2" (at 189.23 76.835 0) (fields_autoplaced)
+    (effects (font (size 1.27 1.27)) (justify left bottom))
+  )
+  (label "cm_out_2" (at 189.23 74.295 0) (fields_autoplaced)
+    (effects (font (size 1.27 1.27)) (justify left bottom))
+  )
   (label "SWCLK" (at 165.735 22.86 180) (fields_autoplaced)
     (effects (font (size 1.27 1.27)) (justify right bottom))
   )
+  (label "SWDIO" (at 188.595 89.535 0) (fields_autoplaced)
+    (effects (font (size 1.27 1.27)) (justify left bottom))
+  )
+  (label "in_3" (at 189.23 66.675 0) (fields_autoplaced)
+    (effects (font (size 1.27 1.27)) (justify left bottom))
+  )
+  (label "cm_out_3" (at 189.23 79.375 0) (fields_autoplaced)
+    (effects (font (size 1.27 1.27)) (justify left bottom))
+  )
+  (label "in_2" (at 189.23 64.135 0) (fields_autoplaced)
+    (effects (font (size 1.27 1.27)) (justify left bottom))
+  )
   (label "SWDIO" (at 165.735 20.32 180) (fields_autoplaced)
+    (effects (font (size 1.27 1.27)) (justify right bottom))
+  )
+  (label "cm_out_1" (at 189.23 69.215 0) (fields_autoplaced)
+    (effects (font (size 1.27 1.27)) (justify left bottom))
+  )
+  (label "SWCLK" (at 188.595 86.995 0) (fields_autoplaced)
+    (effects (font (size 1.27 1.27)) (justify left bottom))
+  )
+  (label "vm_out_3" (at 139.7 69.215 180) (fields_autoplaced)
+    (effects (font (size 1.27 1.27)) (justify right bottom))
+  )
+  (label "vm_out_2" (at 139.7 66.675 180) (fields_autoplaced)
+    (effects (font (size 1.27 1.27)) (justify right bottom))
+  )
+  (label "rs485-tx" (at 189.23 81.915 0) (fields_autoplaced)
+    (effects (font (size 1.27 1.27)) (justify left bottom))
+  )
+  (label "rs485-de" (at 139.7 76.835 180) (fields_autoplaced)
     (effects (font (size 1.27 1.27)) (justify right bottom))
   )
@@
     )
   )
-  (symbol (lib_id "power:+3.3V") (at 137.795 74.93 0) (unit 1)
-    (in_bom yes) (on_board yes) (dnp no) (fields_autoplaced)
-    (property "Reference" "#PWR01" (at 137.795 78.74 0)
-      (effects (font (size 1.27 1.27)) hide)
-    )
-    (property "Value" "+3.3V" (at 137.795 71.12 0)
+  (symbol (lib_id "power:+3.3V") (at 164.465 53.975 0) (unit 1)
+    (in_bom yes) (on_board yes) (dnp no) (fields_autoplaced)
+    (property "Reference" "#PWR01" (at 164.465 57.785 0)
+      (effects (font (size 1.27 1.27)) hide)
+    )
+    (property "Value" "+3.3V" (at 164.465 50.165 0)
       (effects (font (size 1.27 1.27)))
     )
-    (property "Footprint" "" (at 137.795 74.93 0)
-      (effects (font (size 1.27 1.27)) hide)
-    )
-    (property "Datasheet" "" (at 137.795 74.93 0)
+    (property "Footprint" "" (at 164.465 53.975 0)
+      (effects (font (size 1.27 1.27)) hide)
+    )
+    (property "Datasheet" "" (at 164.465 53.975 0)
       (effects (font (size 1.27 1.27)) hide)
     )
@@
     )
   )
-  (symbol (lib_id "MCU_ST_STM32G0:STM32G030F6Px") (at 137.795 97.79 0) (unit 1)
-    (in_bom yes) (on_board yes) (dnp no) (fields_autoplaced)
-    (property "Reference" "U1" (at 139.7509 76.2 0)
-      (effects (font (size 1.27 1.27)) (justify left))
-    )
-    (property "Value" "STM32G030F6Px" (at 139.7509 78.74 0)
-      (effects (font (size 1.27 1.27)) (justify left))
-    )
-    (property "Footprint" "Package_SO:TSSOP-20_4.4x6.5mm_P0.65mm" (at 120.015 115.57 0)
+  (symbol (lib_id "Device:C") (at 40.64 33.02 0) (unit 1)
+    (in_bom yes) (on_board yes) (dnp no) (fields_autoplaced)
+    (property "Reference" "C1" (at 44.45 32.385 0)
+      (effects (font (size 1.27 1.27)) (justify left))
+    )
+    (property "Value" "C" (at 44.45 34.925 0)
+      (effects (font (size 1.27 1.27)) (justify left))
+    )
+    (property "Footprint" "" (at 41.6052 36.83 0)
+      (effects (font (size 1.27 1.27)) hide)
+    )
+    (property "Datasheet" "~" (at 40.64 33.02 0)
+      (effects (font (size 1.27 1.27)) hide)
+    )
+    (pin "1")
+    (pin "2")
+    (instances
+      (project "in-out-port"
+        (path "/e0db4e7e-6f46-4ab1-9056-75c76d7da36a"
+          (reference "C1") (unit 1)
+        )
+      )
+    )
+  )
+  (symbol (lib_id "MCU_ST_STM32G0:STM32G030F6Px") (at 164.465 76.835 0) (unit 1)
+    (in_bom yes) (on_board yes) (dnp no) (fields_autoplaced)
+    (property "Reference" "U1" (at 166.4209 55.245 0)
+      (effects (font (size 1.27 1.27)) (justify left))
+    )
+    (property "Value" "STM32G030F6Px" (at 166.4209 57.785 0)
+      (effects (font (size 1.27 1.27)) (justify left))
+    )
+    (property "Footprint" "Package_SO:TSSOP-20_4.4x6.5mm_P0.65mm" (at 146.685 94.615 0)
       (effects (font (size 1.27 1.27)) (justify right) hide)
     )
-    (property "Datasheet" "https://www.st.com/resource/en/datasheet/stm32g030f6.pdf" (at 137.795 97.79 0)
+    (property "Datasheet" "https://www.st.com/resource/en/datasheet/stm32g030f6.pdf" (at 164.465 76.835 0)
       (effects (font (size 1.27 1.27)) hide)
     )
@@
     )
   )
-  (symbol (lib_id "power:GND") (at 137.795 120.015 0) (unit 1)
-    (in_bom yes) (on_board yes) (dnp no) (fields_autoplaced)
-    (property "Reference" "#PWR03" (at 137.795 126.365 0)
-      (effects (font (size 1.27 1.27)) hide)
-    )
-    (property "Value" "GND" (at 137.795 124.46 0)
+  (symbol (lib_id "power:GND") (at 164.465 99.06 0) (unit 1)
+    (in_bom yes) (on_board yes) (dnp no) (fields_autoplaced)
+    (property "Reference" "#PWR03" (at 164.465 105.41 0)
+      (effects (font (size 1.27 1.27)) hide)
+    )
+    (property "Value" "GND" (at 164.465 103.505 0)
       (effects (font (size 1.27 1.27)))
     )
-    (property "Footprint" "" (at 137.795 120.015 0)
-      (effects (font (size 1.27 1.27)) hide)
-    )
-    (property "Datasheet" "" (at 137.795 120.015 0)
-      (effects (font (size 1.27 1.27)) hide)
-    )
+    (property "Footprint" "" (at 164.465 99.06 0)
+      (effects (font (size 1.27 1.27)) hide)
+    )
+    (property "Datasheet" "" (at 164.465 99.06 0)
+      (effects (font (size 1.27 1.27)) hide)
+    )

Commit message: updated Schematic
Parts:
- added D1: D_Zener, symbol Device:D_Zener
- added D2, D3, D4: Schottky, symbol Device:D_Schottky
- added J2: OUT, symbol Connector:Screw_Terminal_01x06
- added J3: IN, symbol Connector:Screw_Terminal_01x06
- added Q1: BC856BS, Package_TO_SOT_SMD:SOT-363_SC-70-6, symbol Transistor_BJT:BC856BS
- added Q2: BC846BS, Package_TO_SOT_SMD:SOT-363_SC-70-6, symbol Transistor_BJT:BC846BS
- added Q4: Q_PMOS_GDS, symbol Device:Q_PMOS_GDS
- added R1: 100k, symbol Device:R
- added R2, R3, R5: 1k, symbol Device:R
- added R4: 10k, symbol Device:R
- added RShunt: 5m, symbol Device:R
- added SW1: PWM-SCHOTTKY, symbol Switch:SW_DIP_x03
Connections:
- net GND: now also D2.2 (A), D3.2 (A), D4.2 (A), J2.4 (Pin_4), J2.5 (Pin_5), J2.6 (Pin_6), J3.4 (Pin_4), J3.5 (Pin_5), J3.6 (Pin_6), R2.2, R3.2, R5.2
- new net: Q1.3 (C2), Q2.2 (B1), Q2.3 (C2), Q2.5 (B2)
- new net: Q1.4 (E2), R1.2
- new net: Q1.2 (B1), Q1.5 (B2), Q1.6 (C1), Q2.6 (C1)
- new net: D3.1 (K), SW1.5
- new net: Q2.1 (E1), R3.1
- new net: D4.1 (K), SW1.6
- new net: D2.1 (K), SW1.4
- new net IN_1: J3.1 (Pin_1)
- new net IN_2: J3.2 (Pin_2)
- new net IN_3: J3.3 (Pin_3)
- new net MOS-SOURCE: D1.1 (K), Q1.1 (E1), Q4.3 (S), RShunt.2
- new net drive_mos: D1.2 (A), Q4.1 (G)
- new net load: Q4.2 (D), R4.1
- new net load_1: J2.1 (Pin_1), SW1.1
- new net load_2: J2.2 (Pin_2), SW1.2
- new net load_3: J2.3 (Pin_3), SW1.3
- new net mc: Q2.4 (E2), R2.1
- new net mv: R4.2, R5.1
- new net source: R1.1, RShunt.1
Other:
- note added: "for every output"

Commit message: updated Schematic
Parts:
- removed D1: D_Zener, symbol Device:D_Zener
- removed Q1: BC856BS, Package_TO_SOT_SMD:SOT-363_SC-70-6, symbol Transistor_BJT:BC856BS
- added D1: 1N4148WS, Diode_SMD:D_SOD-323, symbol Diode:1N4148WS
- added D5: D_Zener, symbol Device:D_Zener
- added Q1: PNP, symbol Simulation_SPICE:PNP
- added R6: 1k, symbol Device:R
- added U2: ~, Package_TO_SOT_SMD:SOT-363_SC-70-6, symbol lib:TP181
- added U3: ZXGD3009E6, Package_TO_SOT_SMD:SOT-23-6, symbol Driver_FET:ZXGD3009E6
- C1: value C -> 100n
- R1: value 100k -> 10k
- R3: value 1k -> 10k
Connections:
- net +3.3V: now also U2.3 (V+)
- net GND: now also C1.2, Q2.4 (E2), R1.2, Q1.1 (C), U2.1 (REF), U2.2 (GND); no longer R2.2, R3.2
- net MOS-SOURCE: now also U2.5 (IN-)
- net drive_mos: now also U3.4 (SINK), U3.6 (SOURCE)
- net mc: now also U2.6 (OUT); no longer Q2.4 (E2), R2.1
- net out_1: now also R6.1
- net at Q2.6 (C1): now also R2.2, U3.2 (IN)
- net +36V: now reaches R3.1
- net +36V: now also R2.1, RShunt.1, D5.1 (K), U2.4 (IN+), U3.1 (VCC); no longer Q2.1 (E1)
- net pmos-gate-sply: now reaches C1.1
- net pmos-gate-sply: now also Q2.1 (E1), Q1.3 (E), U3.3 (VEE)
- net source: no longer names the net of R1.1
- net source: now also D5.2 (A), Q1.2 (B); no longer RShunt.1
- new net: D1.2 (A), Q2.3 (C2), R3.2
- new net: D1.1 (K), Q2.2 (B1)
- new net: Q2.5 (B2), R6.2
Other:
- note added: "power supply in max 36V to 3.3V"
- note removed: "power supply in max 35V to 3.3V"
- moved on the sheet: C1, Q4, R4, R5

Commit message: updated Schematic
Parts:
- added C2, C3, C4: 100n, symbol Device:C
- added C5: 1u, symbol Device:C
- added D10, D11, D12: LED, symbol Device:LED
- added D6, D7, D8, D9: 1N4148WS, Diode_SMD:D_SOD-323, symbol Diode:1N4148WS
- added J4: POWER, symbol Connector:Screw_Terminal_01x02
- added Q3, Q6: BC846BS, Package_TO_SOT_SMD:SOT-363_SC-70-6, symbol Transistor_BJT:BC846BS
- added Q5, Q7: Q_PMOS_GDS, symbol Device:Q_PMOS_GDS
- added R10, R13, R15, R21, R22, R23, R24, R26, R28, R30, R31, R32, R8: 10k, Resistor_SMD:R_0805_2012Metric, symbol Device:R
- added R11, R12, R14, R16, R17, R18, R19, R20, R25, R27, R29, R7, R9: 1k, Resistor_SMD:R_0805_2012Metric, symbol Device:R
- added RShunt1, RShunt2: 5m, symbol Device:R
- added SW2: ANA/DIG, symbol Switch:SW_DIP_x06
- added SW3: RESET, symbol Switch:SW_Push
- added U4, U6: ~, Package_TO_SOT_SMD:SOT-363_SC-70-6, symbol lib:TP181
- added U5, U7: ZXGD3009E6, Package_TO_SOT_SMD:SOT-23-6, symbol Driver_FET:ZXGD3009E6
- added U8, U9: LM358, symbol Amplifier_Operational:LM358
- R2, R3, R4, R5, R6: footprint (none) -> Resistor_SMD:R_0805_2012Metric
Connections:
- net load is gone; now on net load_1: Q4.2 (D), R4.1
- net +3.3V: now also C2.1, C4.2, R17.1, U4.3 (V+), U6.3 (V+), U8.8 (V+), U9.8 (V+)
- net +36V: now also J4.1 (Pin_1), R13.1, R14.1, R8.1, R9.1, RShunt1.1, RShunt2.1, U4.4 (IN+), U5.1 (VCC), U6.4 (IN+), U7.1 (VCC)
- net GND: now also C2.2, C3.1, C4.1, C5.2, D10.1 (K), D11.1 (K), D12.1 (K), D9.1 (K), J4.2 (Pin_2), Q3.4 (E2), Q6.4 (E2), R11.2, R16.2, R25.2, R27.2, R29.2, SW3.1, U4.1 (REF), U4.2 (GND), U6.1 (REF), U6.2 (GND), U8.4 (V-), U9.4 (V-)
- net IN_1: now also R24.1
- net IN_2: now also R26.1
- net IN_3: now also R28.1
- net MOS-SOURCE: now also Q5.3 (S), Q7.3 (S), RShunt1.2, RShunt2.2, U4.5 (IN-), U6.5 (IN-)
- net in_1: now also SW2.12, SW2.2
- net in_2: now also SW2.10, SW2.4
- net in_3: now also SW2.6, SW2.8
- net load_1: now also R31.1
- net load_2: now also Q5.2 (D), R10.1, R30.1
- net load_3: now also Q7.2 (D), R15.1, R32.1
- net out_2: now also R7.1
- net out_3: now also R12.1
- net pmos-gate-sply: now also C5.1, Q3.1 (E1), Q6.1 (E1), U5.3 (VEE), U7.3 (VEE)
- net at U1.6 (NRST): now also SW3.2
- net drive_mos renamed drive_mos_1
- net mc renamed mc_1
- net mv renamed mv_1
- new net: R18.2, R21.1, U8.3 (+)
- new net: Q6.6 (C1), R14.2, U7.2 (IN)
- new net: D8.1 (K), D9.2 (A)
- new net: D11.2 (A), R31.2
- new net: D6.2 (A), Q3.3 (C2), R8.2
- new net: Q3.5 (B2), R7.2
- new net: R20.2, R23.1, U9.3 (+)
- new net: D12.2 (A), R32.2
- new net: D6.1 (K), Q3.2 (B1)
- new net: Q3.6 (C1), R9.2, U5.2 (IN)
- new net: R19.2, R22.1, U8.5 (+)
- new net: D7.2 (A), Q6.3 (C2), R13.2
- new net: D7.1 (K), Q6.2 (B1)
- new net: Q6.5 (B2), R12.2
- new net: D10.2 (A), R30.2
- new net drive_mos_2: Q5.1 (G), U5.4 (SINK), U5.6 (SOURCE)
- new net drive_mos_3: Q7.1 (G), U7.4 (SINK), U7.6 (SOURCE)
- new net in_1_1: R18.1, R24.2, R25.1, SW2.1
- new net in_1_2: R21.2, SW2.11, U8.1
- new net in_2_1: R19.1, R26.2, R27.1, SW2.3
- new net in_2_2: R22.2, SW2.9, U8.7
- new net in_3_1: R20.1, R28.2, R29.1, SW2.5
- new net in_3_2: R23.2, SW2.7, U9.1
- new net mc_2: U4.6 (OUT)
- new net mc_3: U6.6 (OUT)
- new net mv_2: R10.2, R11.1
- new net mv_3: R15.2, R16.1
- new net vref_schmitt: C3.2, D8.2 (A), R17.2, U8.2 (-), U8.6 (-), U9.2 (-)
Other:
- note added: "ANALOG/DIGITAL INPUT"
- note added: "Alternative MCU: STM32G030K8T6 (LQFP32) STM32G030C8T6 (LQFP48)"
- note added: "OPTIONAL"
- note added: "OUTPUT 1"
- note added: "OUTPUT 2"
- note added: "OUTPUT 3"
- note added: "todo: power supply in max 36V to 3.3V"
- note removed: "for every output"
- note removed: "power supply in max 36V to 3.3V"
- company: (none) -> Philipp Schnecker
- title: (none) -> ModSmart-IOUnit
- moved on the sheet: C1, D1, D2, D3, D4, D5, J1, J2, J3, Q1, Q2A, Q2B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

Commit message: updated Schematic
Parts:
- added C6: 100n, symbol Device:C
- added R33, R34, R35, R38, R39: 1k, Resistor_SMD:R_0805_2012Metric, symbol Device:R
- added R36, R37: 10k, Resistor_SMD:R_0805_2012Metric, symbol Device:R
- added U10: 4072, symbol 4xxx:4072
- added U11, U12: LM358, symbol Amplifier_Operational:LM358
Connections:
- net +3.3V: now also C6.2, U11.8 (V+), U12.8 (V+)
- net GND: now also C6.1, R39.2, U11.4 (V-), U12.4 (V-)
- net in_2_1: now also R34.1
- net mc_1: now also R35.1
- new net: R33.1, R38.2, R39.1
- new net: R33.2, R36.1, U11.3 (+)
- new net: R35.2, U12.3 (+)
- new net: R38.1, U12.1, U12.2 (-)
- new net: R34.2, R37.1, U11.5 (+)
- new net oc_int: U10.1
- new net or1: R36.2, U10.2, U11.1
- new net or2: R37.2, U10.3, U11.7
- new net or3: U10.4
- new net vref_oc: U11.2 (-), U11.6 (-)
Other:
- note added: "Over current detection and schmitt-trigger and buffer for mcu measurement. replace op amp wit RRIO op amp"
